Commit message: Changes made to state publisher and urdf

File: my_2d_robot/urdf/my2drobo.urdf (robot description, URDF)
Before this commit: robot robo_2d, 4 links, 3 joints
Links:
- link base: geometry visual box size=0.0 0.0 0.0
- link link1: geometry visual box size=5 0.25 1
- link link2: geometry visual box size=5 0.25 1
Joints:
- joint end_effector: origin xyz=0.0 0.0 0.0 -> xyz=2.5 0.0 0.0
- joint joint1: origin xyz=0.025 0.0 0.1 rpy=0.0 0.0 0.0 -> xyz=0.0 0.0 0.0 rpy=0.0 0.0 0.0
- joint joint2: origin xyz=-0.025 0.0 0.4 rpy=0.0 0.0 0.0 -> xyz=5 0.0 0.0 rpy=0.0 0.0 0.0

Commit message: changes made for testing

File: my_2d_robot/urdf/my2drobo.urdf (robot description, URDF)
Before this commit: robot robo_2d, 4 links, 3 joints
Joints:
- joint joint1: axis 0.0 1 0.0 -> 0.0 -1 0.0
- joint joint2: axis 0.0 1 0.0 -> 0.0 -1 0.0

Commit message: State publisher (#4)
* First_attempt_at_URDF

* First_attempt_at_URDF

* Ignoring robo_2d.pdf

* Uploading the created package with URDf

* changed axis of rotation

* updated .gitignore

* New line included

* state_publisher first try

* first attempt -Cmake errors

* first attempt -Cmake errors

* Changes made to CMakeLists.txt, my_2d_robo_state_publisher and launch file to fix cmake and roslaunch errors

* Changes made to state publisher and urdf

* Comment modified in state publisher

* Subscriber node

* Modifications made to CMakeLists and subscriber files

* Modifications made to CMakeLists and subscriber files

* Minor changes made to CMakeLists, state publisher and urdf

* Minor changes made to CMakeLists, state publisher and urdf

* Changes made for PR except last change (debug mode flag)

* Slightly fleshed out readme

* changes made to state publisher and rviz files

* changes made to launch file and state publisher to include full range of motion and set the loop rate in the launch file

* Fixed angle conventon for 2D robot

File: my_2d_robot/urdf/my2drobo.urdf (robot description, URDF)
Before this commit: robot robo_2d, 4 links, 3 joints
Links:
- link base: geometry visual box size=0.0 0.0 0.0
- link link1: geometry visual box size=5 0.25 1
- link link2: geometry visual box size=5 0.25 1
Joints:
- joint end_effector: origin xyz=0.0 0.0 0.0 rpy=0.0 0.0 0.0 -> xyz=2.5 0.0 0.0
- joint joint1: axis 0.0 1 0.0 -> 0.0 -1 0.0; origin xyz=0.025 0.0 0.1 rpy=0.0 0.0 0.0 -> xyz=0.0 0.0 0.0 rpy=0.0 0.0 0.0
- joint joint2: axis 0.0 1 0.0 -> 0.0 -1 0.0; origin xyz=-0.025 0.0 0.4 rpy=0.0 0.0 0.0 -> xyz=5 0.0 0.0 rpy=0.0 0.0 0.0
